File: KiCad/beepy.kicad_pcb (KiCad board)
At the start: 2 copper layers, 74 x 104 mm, 160 parts, among them J1 FDX0019B1, J10 FDX0019B1, J11 FDX0019B1, J12 FDX0019B1, J13 FDX0019B1, J14 FDX0019B1, J15 USB_C_Receptacle_USB2.0, J16 FDX0019B1, J17 FDX0019B1, J18 FDX0019B1, J19 FDX0019B1, J2 FDX0019B1, J20 FDX0019B1, J21 FDX0019B1, J23 FDX0019B1, J24 FDX0019B1, J25 FDX0019B1, J26 FDX0019B1, J27 FDX0019B1, J28 FDX0019B1, J29 FDX0019B1, J3 FDX0019B1, J30 FDX0019B1, J31 FDX0019B1, J32 FDX0019B1, J33 FDX0019B1, J34 FDX0019B1, J35 FDX0019B1, J36 FDX0019B1, J37 FDX0019B1, J38 FDX0019B1, J39 FDX0019B1, J4 FDX0019B1, J40 FDX0019B1, J41 FDX0019B1, J42 FDX0019B1, J43 Battery, J44 Header 1, J45 PRG_HEADER, J46 Header 2, J47 Header 3, J5 FDX0019B1, J6 FDX0019B1, J7 FDX0019B1, J8 FDX0019B1, J9 FDX0019B1, M1 MountingHole_2.5mm_Pad, M2 MountingHole_2.5mm_Pad, M3 MountingHole_2.5mm_Pad, M4 MountingHole_2.5mm_Pad, Q1 SI2301, Q2 SI2301, Q3 BSS138, Q4 BSS138, Q5 BSS138, Q6 BSS138, Q7 BSS138, Q8 BSS138, Q9 S8050, SW1 ON/OFF, SW2 Button, U1 TP4054, U2 TPS61090, U3 LS027B7DH01, U4 AP2112K-3.3, U5 GD25Q16xS, U6 RP2040, U7 ME6212C18M5G, U8 ME6212C28M5G, U9 BBQ20KBD, Y1 XYDBPCNANF-12MHZ

Commit message: updated pcb, second checks, gerbers
Parts:
- moved G*** 8.28 mm to (83.5, 111.5)
Routing:
- net GND: track 107.5 -> 126.0 mm
- net +5V: track 230.3 -> 231.9 mm
Other:
- board text added: "Designed by SQFMI"
- board text added: "Second life by"
- board text added: "archFX"
- board text added: "archfx.github.io"
- board text removed: "SQFMI"
- board text removed: "x"
Changed lines of the file:
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@@
 	(footprint "beepy:beepy_logo_2"
 		(layer "B.Cu")
-		(at 82.915347 119.76 180)
+		(at 83.5 111.5 180)
 		(property "Reference" "G***"
 			(at 0 0 0)
@@
 		(layer "F.Fab")
 	)
-	(gr_text "x"
-		(at 82.91 115.86 0)
+	(gr_text "archFX"
+		(at 92.5 120 0)
 		(layer "B.Cu")
 		(effects
 			(font
-				(size 1.5 1.5)
-				(thickness 0.3)
+				(size 4 4)
+				(thickness 1)
+				(bold yes)
 			)
-			(justify mirror)
-		)
-	)
-	(gr_text "SQFMI"
-		(at 82.893674 112.159721 0)
-		(layer "B.Cu")
-		(effects
-			(font
-				(size 3 3)
-				(thickness 0.6)
-			)
-			(justify mirror)
+			(justify left bottom mirror)
 		)
 	)
@@
 		)
 	)
+	(gr_text "archfx.github.io"
+		(at 83.5 121.5 0)
+		(layer "B.SilkS" knockout)
+		(effects
+			(font
+				(size 1 1)
+				(thickness 0.12)
+			)
+			(justify left bottom mirror)
+		)
+	)
+	(gr_text "Second life by"
+		(at 95 115.5 0)
+		(layer "B.SilkS")
+		(effects
+			(font
+				(size 1 1)
+				(thickness 0.15)
+			)
+			(justify left bottom mirror)
+		)
+	)
 	(gr_text "+"
 		(at 96.9 136.47 0)
@@
 		)
 	)
+	(gr_text "Designed by SQFMI"
+		(at 95 109 0)
+		(layer "B.SilkS")
+		(effects
+			(font
+				(size 0.7 0.7)
+				(thickness 0.15)
+				(bold yes)
+			)
+			(justify left bottom mirror)
+		)
+	)
 	(gr_text "."
 		(at 74.15 129.33 0)
@@
 		)
 	)
+	(gr_text "archFX"
+		(at 92.5 120 0)
+		(layer "B.SilkS")
+		(effects
+			(font
+				(size 4 4)
+				(thickness 1)
+				(bold yes)
+			)
+			(justify left bottom mirror)
+		)
+	)
 	(gr_text "M2"
 		(at 120.08 46.27 0)
@@
 		)
 	)
-	(gr_text "SQFMI"
-		(at 82.91 112.14 0)
-		(layer "B.Mask")
-		(effects
-			(font
-				(size 3 3)
-				(thickness 0.6)
-			)
-			(justify mirror)
-		)
-	)
-	(gr_text "x"
-		(at 82.91 115.86 0)
-		(layer "B.Mask")
-		(effects
-			(font
-				(size 1.5 1.5)
-				(thickness 0.3)
-			)
-			(justify mirror)
-		)
-	)
 	(gr_text "REF**"
 		(locked yes)
@@
 		(net 1)
 	)
+	(segment
+		(start 106.5022 115.7478)
+		(end 106.5022 113.8174)
+		(width 0.2)
+		(layer "F.Cu")
+		(net 1)
+	)
+	(segment
+		(start 106.5022 113.8174)
+		(end 105.5116 112.8268)
+		(width 0.2)
+		(layer "F.Cu")
+		(net 1)
+	)
 	(via
 		(at 115.39 109.01)
@@
 	)
 	(segment
+		(start 78.57563 69.343)
+		(end 80.72963 69.343)
+		(width 0.4)
+		(layer "B.Cu")
+		(net 1)
+	)
+	(segment
 		(start 65.935 126.33)
 		(end 64.68 126.33)
@@
 	)
 	(segment
+		(start 80.72963 69.343)
+		(end 81 69.61337)
+		(width 0.4)
+		(layer "B.Cu")
+		(net 1)
+	)
+	(segment
 		(start 116.71 124.595)
 		(end 117.715 124.595)
@@
 	)
 	(segment
+		(start 81 75.032)
+		(end 81.968 76)
+		(width 0.4)
+		(layer "B.Cu")
+		(net 1)
+	)
+	(segment
 		(start 67.17375 84.04)
 		(end 67.77445 84.04)
@@
 	)
 	(segment
+		(start 77.122104 67.48)
+		(end 77.122104 67.889474)
+		(width 0.4)
+		(layer "B.Cu")
+		(net 1)
+	)
+	(segment
 		(start 70.2825 134.1)
 		(end 71.2575 133.125)
@@
 	)
 	(segment
+		(start 81 69.61337)
+		(end 81 75.032)
+		(width 0.4)
+		(layer "B.Cu")
+		(net 1)
+	)
+	(segment
 		(start 89.34 81.7575)
 		(end 88.84 81.7575)
@@
 	)
 	(segment
+		(start 81.968 76)
+		(end 81.968 77.491332)
+		(width 0.4)
+		(layer "B.Cu")
+		(net 1)
+	)
+	(segment
 		(start 70.894002 71.5175)
 		(end 70.876502 71.5)
@@
 	)
 	(segment
+		(start 77.122104 67.889474)
+		(end 78.57563 69.343)
+		(width 0.4)
+		(layer "B.Cu")
+		(net 1)
+	)
+	(segment
 		(start 109.72 101.27875)
 		(end 109.72 102.32)
@@
 	)
 	(segment
+		(start 81.968 77.491332)
+		(end 82.926668 78.45)
+		(width 0.4)
+		(layer "B.Cu")
+		(net 1)
+	)
+	(segment
 		(start 104.143911 135.826)
 		(end 104.143911 134.953911)
@@
 	)
 	(segment
+		(start 82.926668 78.45)
+		(end 83.48 78.45)
+		(width 0.4)
+		(layer "B.Cu")
+		(net 1)
+	)
+	(segment
 		(start 106.185 116.22)
 		(end 105.33 116.22)
@@
 	)
 	(via
-		(at 74.3712 84.2264)
-		(size 0.5)
-		(drill 0.3)
+		(at 74 84.2264)
+		(size 1)
+		(drill 0.4)
 		(layers "F.Cu" "B.Cu")
 		(net 10)
 	)
 	(via
-		(at 72.0344 91.948)
-		(size 0.5)
-		(drill 0.3)
+		(at 74 91.5)
+		(size 1)
+		(drill 0.4)
 		(layers "F.Cu" "B.Cu")
 		(net 10)
@@
 	)
 	(segment
-		(start 74.59 84.0076)
-		(end 74.3712 84.2264)
-		(width 0.127)
-		(layer "B.Cu")
-		(net 10)
-	)
-	(segment
 		(start 66.6 125.38)
 		(end 67.08 125.86)
@@
 	)
 	(segment
-		(start 72.2376 91.7448)
-		(end 72.0344 91.948)
-		(width 0.127)
-		(layer "B.Cu")
-		(net 10)
-	)
-	(segment
 		(start 90.84 81.7625)
 		(end 89.84 81.7625)
@@
 	)
 	(segment
-		(start 61.5696 91.948)
-		(end 63.0428 91.948)
-		(width 0.127)
+		(start 66.59 127.28)
+		(end 67.08 126.79)
+		(width 0.25)
 		(layer "B.Cu")
 		(net 10)
 	)
 	(segment
-		(start 66.59 127.28)
-		(end 67.08 126.79)
-		(width 0.25)
+		(start 61.1216 91.5)
+		(end 57.912 88.2904)
+		(width 0.127)
 		(layer "B.Cu")
 		(net 10)
@@
 	)
 	(segment
-		(start 74.59 81.35)
-		(end 74.59 84.0076)
-		(width 0.127)
-		(layer "B.Cu")
-		(net 10)
-	)
-	(segment
 		(start 74.34 79.115)
 		(end 74.34 81.1)
@@
 	)
 	(segment
+		(start 74 84.2264)
+		(end 74.59 83.6364)
+		(width 0.127)
+		(layer "B.Cu")
+		(net 10)
+	)
+	(segment
 		(start 68.2625 125.4125)
 		(end 68.2625 121.5675)
@@
 	)
 	(segment
+		(start 74.59 83.6364)
+		(end 74.59 81.35)
+		(width 0.127)
+		(layer "B.Cu")
+		(net 10)
+	)
+	(segment
 		(start 82.695 76.9925)
 		(end 83.4675 76.9925)
@@
 	(segment
 		(start 57.912 88.2904)
-		(end 61.5696 91.948)
-		(width 0.127)
-		(layer "B.Cu")
-		(net 10)
-	)
-	(segment
-		(start 63.0428 91.948)
-		(end 72.0344 91.948)
+		(end 57.912 77.102)
 		(width 0.127)
 		(layer "B.Cu")
@@
 	)
 	(segment
-		(start 57.912 77.102)
-		(end 57.912 88.2904)
-		(width 0.127)
+		(start 126.04 77.87)
+		(end 122.04 77.87)
+		(width 0.2)
 		(layer "B.Cu")
 		(net 10)
 	)
 	(segment
-		(start 126.04 77.87)
-		(end 122.04 77.87)
-		(width 0.2)
+		(start 57.912 77.102)
+		(end 56.14 75.33)
+		(width 0.127)
 		(layer "B.Cu")
 		(net 10)
@@
 	)
 	(segment
-		(start 68.2625 121.3425)
-		(end 68.2625 121.3525)
-		(width 0.4)
+		(start 74 91.5)
+		(end 61.1216 91.5)
+		(width 0.127)
 		(layer "B.Cu")
 		(net 10)
 	)
 	(segment
-		(start 56.14 75.33)
-		(end 57.912 77.102)
-		(width 0.127)
+		(start 68.2625 121.3425)
+		(end 68.2625 121.3525)
+		(width 0.4)
 		(layer "B.Cu")
 		(net 10)
