File: KiCad/beepy.kicad_sch (KiCad schematic)
At the start: 102 parts, among them J1 FDX0019B1, J10 FDX0019B1, J11 FDX0019B1, J12 FDX0019B1, J13 FDX0019B1, J14 FDX0019B1, J15 USB_C_Receptacle_USB2.0, J16 FDX0019B1, J17 FDX0019B1, J18 FDX0019B1, J19 FDX0019B1, J2 FDX0019B1, J20 FDX0019B1, J21 FDX0019B1, J22 Pi Zero, J23 FDX0019B1, J24 FDX0019B1, J25 FDX0019B1, J26 FDX0019B1, J27 FDX0019B1, J28 FDX0019B1, J29 FDX0019B1, J3 FDX0019B1, J30 FDX0019B1, J31 FDX0019B1, J32 FDX0019B1, J33 FDX0019B1, J34 FDX0019B1, J35 FDX0019B1, J36 FDX0019B1, J37 FDX0019B1, J38 FDX0019B1, J39 FDX0019B1, J4 FDX0019B1, J40 FDX0019B1, J41 FDX0019B1, J42 FDX0019B1, J43 Battery, J44 Header 1, J45 PRG_HEADER, J46 Header 2, J47 Header 3, J5 FDX0019B1, J6 FDX0019B1, J7 FDX0019B1, J8 FDX0019B1, J9 FDX0019B1, Q1 SI2301, Q2 SI2301, Q9 S8050, SW1 ON/OFF, SW2 Button, U1 TP4054, U2 TPS61090, U3 LS027B7DH01

Commit message: BoM added
Parts:
- C3: value 22uF -> 2.2uF
Changed lines of the file:
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@@
 		(fields_autoplaced yes)
 		(property "Reference" "C3"
-			(at 182.499 143.7639 0)
+			(at 181.61 143.7639 0)
 			(effects
 				(font
@@
 			)
 		)
-		(property "Value" "22uF"
-			(at 182.499 146.3039 0)
+		(property "Value" "2.2uF"
+			(at 181.61 146.3039 0)
 			(effects
 				(font
